Commit message: Add reproducible Gazebo LeRobot dataset collection

File: open_manipulator_description/ros2_control/omx_f.ros2_control.xacro (robot description, xacro)
@@ -64,9 +64,7 @@
       <xacro:if value="$(arg use_sim)">
         <joint name="${prefix}gripper_joint_2">
-          <param name="mimic">${prefix}gripper_joint_1</param>
-          <param name="multiplier">-1</param>
+          <command_interface name="position"/>
           <state_interface name="position"/>
           <state_interface name="velocity"/>
-          <state_interface name="effort"/>
         </joint>
       </xacro:if>

File: open_manipulator_description/urdf/omx_f/omx_f.urdf.xacro (robot description, xacro)
@@ -33,5 +33,5 @@
     </visual>
   </link>
-  <xacro:omx_f prefix="$(arg prefix)" />
+  <xacro:omx_f prefix="$(arg prefix)" use_sim="$(arg use_sim)" />
   <xacro:omx_f_gazebo prefix="$(arg prefix)" />
   <xacro:omx_f_system

File: open_manipulator_description/urdf/omx_f/omx_f_arm.urdf.xacro (robot description, xacro)
@@ -1,5 +1,5 @@
 <?xml version="1.0" encoding="UTF-8"?>
 <robot xmlns:xacro="http://www.ros.org/wiki/xacro">
-   <xacro:macro name="omx_f" params="prefix">
+   <xacro:macro name="omx_f" params="prefix use_sim:=false">
    <xacro:property name="meshes_file_direction" value="package://open_manipulator_description/meshes/omx_f" />
       <link name="${prefix}link0" >
@@ -247,5 +247,10 @@
          <limit velocity="4.8" effort="1000" lower="${-pi*2.0}" upper="${pi*2.0}" />
          <dynamics damping="0.1" />
-         <mimic joint="${prefix}gripper_joint_1" multiplier="-1"/>
+         <!-- Gazebo's selected physics engine does not implement URDF mimic
+              constraints. In simulation both fingers are commanded explicitly
+              through ros2_control; real hardware keeps the mechanical mimic. -->
+         <xacro:unless value="${use_sim}">
+            <mimic joint="${prefix}gripper_joint_1" multiplier="-1"/>
+         </xacro:unless>
       </joint>
       <link name="${prefix}link7" >
